Commit message: Moved copied files into single directory

File: reach_demo/model/motoman_sia20d/motoman_sia20d_macro.xacro (robot description, xacro)
@@ -1,3 +1,6 @@
 <?xml version="1.0" ?>
+<!-- Notice: this file has been modified from its original version
+     Original: https://github.com/ros-industrial/motoman/blob/43be182c9cb4f62806e479b985965886c8603333/motoman_sia20d_support/urdf/sia20d_macro.xacro
+-->
 <robot xmlns:xacro="http://ros.org/wiki/xacro">
   <xacro:macro name="motoman_sia20d" params="prefix">
@@ -6,5 +9,6 @@
       <visual>
         <geometry>
-          <mesh filename="package://reach_demo/model/meshes/sia20d/visual/MOTOMAN_BASE.stl" />
+<!--          <mesh filename="package://motoman_sia20d_support/meshes/sia20d/visual/MOTOMAN_BASE.stl" />-->
+          <mesh filename="package://reach_demo/model/motoman_sia20d/meshes/sia20d/visual/MOTOMAN_BASE.stl" />
         </geometry>
         <material name="blue">
@@ -14,5 +18,6 @@
       <collision>
         <geometry>
-          <mesh filename="package://reach_demo/model/meshes/sia20d/collision/MOTOMAN_BASE.stl" />
+<!--          <mesh filename="package://motoman_sia20d_support/meshes/sia20d/collision/MOTOMAN_BASE.stl" />-->
+          <mesh filename="package://reach_demo/model/motoman_sia20d/meshes/sia20d/collision/MOTOMAN_BASE.stl" />
         </geometry>
         <material name="yellow">
@@ -25,5 +30,6 @@
         <origin rpy="0 0 3.1416" xyz="0 0 0"/>
         <geometry>
-          <mesh filename="package://reach_demo/model/meshes/sia20d/visual/MOTOMAN_AXIS_S.stl"/>
+<!--          <mesh filename="package://motoman_sia20d_support/meshes/sia20d/visual/MOTOMAN_AXIS_S.stl"/>-->
+          <mesh filename="package://reach_demo/model/motoman_sia20d/meshes/sia20d/visual/MOTOMAN_AXIS_S.stl"/>
         </geometry>
         <material name="silver">
@@ -34,5 +40,6 @@
         <origin rpy="0 0 3.1416" xyz="0 0 0"/>
         <geometry>
-          <mesh filename="package://reach_demo/model/meshes/sia20d/collision/MOTOMAN_AXIS_S.stl" />
+<!--          <mesh filename="package://motoman_sia20d_support/meshes/sia20d/collision/MOTOMAN_AXIS_S.stl" />-->
+          <mesh filename="package://reach_demo/model/motoman_sia20d/meshes/sia20d/collision/MOTOMAN_AXIS_S.stl" />
         </geometry>
         <material name="yellow"/>
@@ -43,5 +50,6 @@
         <origin rpy="1.57 3.1416 3.1416" xyz="0 0 0"/>
         <geometry>
-          <mesh filename="package://reach_demo/model/meshes/sia20d/visual/MOTOMAN_AXIS_L.stl"/>
+<!--          <mesh filename="package://motoman_sia20d_support/meshes/sia20d/visual/MOTOMAN_AXIS_L.stl"/>-->
+          <mesh filename="package://reach_demo/model/motoman_sia20d/meshes/sia20d/visual/MOTOMAN_AXIS_L.stl"/>
         </geometry>
         <material name="blue"/>
@@ -50,5 +58,6 @@
         <origin rpy="1.57 3.1416 3.1416" xyz="0 0 0"/>
         <geometry>
-          <mesh filename="package://reach_demo/model/meshes/sia20d/collision/MOTOMAN_AXIS_L.stl"/>
+<!--          <mesh filename="package://motoman_sia20d_support/meshes/sia20d/collision/MOTOMAN_AXIS_L.stl"/>-->
+          <mesh filename="package://reach_demo/model/motoman_sia20d/meshes/sia20d/collision/MOTOMAN_AXIS_L.stl"/>
         </geometry>
         <material name="yellow"/>
@@ -59,5 +68,6 @@
         <origin rpy="0 0 0" xyz="0 0 0"/>
         <geometry>
-          <mesh filename="package://reach_demo/model/meshes/sia20d/visual/MOTOMAN_AXIS_E.stl"/>
+<!--          <mesh filename="package://motoman_sia20d_support/meshes/sia20d/visual/MOTOMAN_AXIS_E.stl"/>-->
+          <mesh filename="package://reach_demo/model/motoman_sia20d/meshes/sia20d/visual/MOTOMAN_AXIS_E.stl"/>
         </geometry>
         <material name="silver"/>
@@ -66,5 +76,6 @@
         <origin rpy="0 0 0" xyz="0 0 0"/>
         <geometry>
-          <mesh filename="package://reach_demo/model/meshes/sia20d/collision/MOTOMAN_AXIS_E.stl"/>
+<!--          <mesh filename="package://motoman_sia20d_support/meshes/sia20d/collision/MOTOMAN_AXIS_E.stl"/>-->
+          <mesh filename="package://reach_demo/model/motoman_sia20d/meshes/sia20d/collision/MOTOMAN_AXIS_E.stl"/>
         </geometry>
         <material name="yellow"/>
@@ -75,5 +86,6 @@
         <origin rpy="1.57 -3.1415 3.1416" xyz="0 0 0"/>
         <geometry>
-          <mesh filename="package://reach_demo/model/meshes/sia20d/visual/MOTOMAN_AXIS_U.stl"/>
+<!--          <mesh filename="package://motoman_sia20d_support/meshes/sia20d/visual/MOTOMAN_AXIS_U.stl"/>-->
+          <mesh filename="package://reach_demo/model/motoman_sia20d/meshes/sia20d/visual/MOTOMAN_AXIS_U.stl"/>
         </geometry>
         <material name="blue"/>
@@ -82,5 +94,6 @@
         <origin rpy="1.57 -3.1415 3.1416" xyz="0 0 0"/>
         <geometry>
-          <mesh filename="package://reach_demo/model/meshes/sia20d/collision/MOTOMAN_AXIS_U.stl"/>
+<!--          <mesh filename="package://motoman_sia20d_support/meshes/sia20d/collision/MOTOMAN_AXIS_U.stl"/>-->
+          <mesh filename="package://reach_demo/model/motoman_sia20d/meshes/sia20d/collision/MOTOMAN_AXIS_U.stl"/>
         </geometry>
         <material name="yellow"/>
@@ -91,5 +104,6 @@
         <origin rpy="0 0 0" xyz="0 0 0"/>
         <geometry>
-          <mesh filename="package://reach_demo/model/meshes/sia20d/visual/MOTOMAN_AXIS_R.stl"/>
+<!--          <mesh filename="package://motoman_sia20d_support/meshes/sia20d/visual/MOTOMAN_AXIS_R.stl"/>-->
+          <mesh filename="package://reach_demo/model/motoman_sia20d/meshes/sia20d/visual/MOTOMAN_AXIS_R.stl"/>
         </geometry>
         <material name="silver"/>
@@ -98,5 +112,6 @@
         <origin rpy="0 0 0" xyz="0 0 0"/>
         <geometry>
-          <mesh filename="package://reach_demo/model/meshes/sia20d/collision/MOTOMAN_AXIS_R.stl"/>
+<!--          <mesh filename="package://motoman_sia20d_support/meshes/sia20d/collision/MOTOMAN_AXIS_R.stl"/>-->
+          <mesh filename="package://reach_demo/model/motoman_sia20d/meshes/sia20d/collision/MOTOMAN_AXIS_R.stl"/>
         </geometry>
         <material name="yellow"/>
@@ -107,5 +122,6 @@
         <origin rpy="-1.57 0 0" xyz="0 0 0"/>
         <geometry>
-          <mesh filename="package://reach_demo/model/meshes/sia20d/visual/MOTOMAN_AXIS_B.stl"/>
+<!--          <mesh filename="package://motoman_sia20d_support/meshes/sia20d/visual/MOTOMAN_AXIS_B.stl"/>-->
+          <mesh filename="package://reach_demo/model/motoman_sia20d/meshes/sia20d/visual/MOTOMAN_AXIS_B.stl"/>
         </geometry>
         <material name="blue"/>
@@ -114,5 +130,6 @@
         <origin rpy="-1.57 0 0" xyz="0 0 0"/>
         <geometry>
-          <mesh filename="package://reach_demo/model/meshes/sia20d/collision/MOTOMAN_AXIS_B.stl"/>
+<!--          <mesh filename="package://motoman_sia20d_support/meshes/sia20d/collision/MOTOMAN_AXIS_B.stl"/>-->
+          <mesh filename="package://reach_demo/model/motoman_sia20d/meshes/sia20d/collision/MOTOMAN_AXIS_B.stl"/>
         </geometry>
         <material name="yellow"/>
@@ -122,5 +139,6 @@
       <visual>
         <geometry>
-          <mesh filename="package://reach_demo/model/meshes/sia20d/visual/MOTOMAN_AXIS_T.stl" />
+<!--          <mesh filename="package://motoman_sia20d_support/meshes/sia20d/visual/MOTOMAN_AXIS_T.stl" />-->
+          <mesh filename="package://reach_demo/model/motoman_sia20d/meshes/sia20d/visual/MOTOMAN_AXIS_T.stl" />
         </geometry>
         <material name="silver"/>
@@ -128,5 +146,6 @@
       <collision>
         <geometry>
-          <mesh filename="package://reach_demo/model/meshes/sia20d/collision/MOTOMAN_AXIS_T.stl" />
+<!--          <mesh filename="package://motoman_sia20d_support/meshes/sia20d/collision/MOTOMAN_AXIS_T.stl" />-->
+          <mesh filename="package://reach_demo/model/motoman_sia20d/meshes/sia20d/collision/MOTOMAN_AXIS_T.stl" />
         </geometry>
         <material name="yellow"/>

File: reach_demo/model/reach_study.xacro (robot description, xacro)
@@ -1,5 +1,5 @@
 <?xml version="1.0" ?>
 <robot name="reach_study" xmlns:xacro="http://ros.org/wiki/xacro">
-  <xacro:include filename="$(find reach_demo)/model/motoman_sia20d_macro.xacro" />
+  <xacro:include filename="$(find reach_demo)/model/motoman_sia20d/motoman_sia20d_macro.xacro" />
   <xacro:motoman_sia20d prefix=""/>
   <link name="reach_object"/>
