Commit message: Merged demo into moveit_reach_plugins package

File: moveit_reach_plugins/demo/model/motoman_sia20d/motoman_sia20d_macro.xacro (robot description, xacro)
@@ -10,5 +10,5 @@
         <geometry>
 <!--          <mesh filename="package://motoman_sia20d_support/meshes/sia20d/visual/MOTOMAN_BASE.stl" />-->
-          <mesh filename="package://reach_demo/model/motoman_sia20d/meshes/sia20d/visual/MOTOMAN_BASE.stl" />
+          <mesh filename="package://moveit_reach_plugins/demo/model/motoman_sia20d/meshes/sia20d/visual/MOTOMAN_BASE.stl" />
         </geometry>
         <material name="blue">
@@ -19,5 +19,5 @@
         <geometry>
 <!--          <mesh filename="package://motoman_sia20d_support/meshes/sia20d/collision/MOTOMAN_BASE.stl" />-->
-          <mesh filename="package://reach_demo/model/motoman_sia20d/meshes/sia20d/collision/MOTOMAN_BASE.stl" />
+          <mesh filename="package://moveit_reach_plugins/demo/model/motoman_sia20d/meshes/sia20d/collision/MOTOMAN_BASE.stl" />
         </geometry>
         <material name="yellow">
@@ -31,5 +31,5 @@
         <geometry>
 <!--          <mesh filename="package://motoman_sia20d_support/meshes/sia20d/visual/MOTOMAN_AXIS_S.stl"/>-->
-          <mesh filename="package://reach_demo/model/motoman_sia20d/meshes/sia20d/visual/MOTOMAN_AXIS_S.stl"/>
+          <mesh filename="package://moveit_reach_plugins/demo/model/motoman_sia20d/meshes/sia20d/visual/MOTOMAN_AXIS_S.stl"/>
         </geometry>
         <material name="silver">
@@ -41,5 +41,5 @@
         <geometry>
 <!--          <mesh filename="package://motoman_sia20d_support/meshes/sia20d/collision/MOTOMAN_AXIS_S.stl" />-->
-          <mesh filename="package://reach_demo/model/motoman_sia20d/meshes/sia20d/collision/MOTOMAN_AXIS_S.stl" />
+          <mesh filename="package://moveit_reach_plugins/demo/model/motoman_sia20d/meshes/sia20d/collision/MOTOMAN_AXIS_S.stl" />
         </geometry>
         <material name="yellow"/>
@@ -51,5 +51,5 @@
         <geometry>
 <!--          <mesh filename="package://motoman_sia20d_support/meshes/sia20d/visual/MOTOMAN_AXIS_L.stl"/>-->
-          <mesh filename="package://reach_demo/model/motoman_sia20d/meshes/sia20d/visual/MOTOMAN_AXIS_L.stl"/>
+          <mesh filename="package://moveit_reach_plugins/demo/model/motoman_sia20d/meshes/sia20d/visual/MOTOMAN_AXIS_L.stl"/>
         </geometry>
         <material name="blue"/>
@@ -59,5 +59,5 @@
         <geometry>
 <!--          <mesh filename="package://motoman_sia20d_support/meshes/sia20d/collision/MOTOMAN_AXIS_L.stl"/>-->
-          <mesh filename="package://reach_demo/model/motoman_sia20d/meshes/sia20d/collision/MOTOMAN_AXIS_L.stl"/>
+          <mesh filename="package://moveit_reach_plugins/demo/model/motoman_sia20d/meshes/sia20d/collision/MOTOMAN_AXIS_L.stl"/>
         </geometry>
         <material name="yellow"/>
@@ -69,5 +69,5 @@
         <geometry>
 <!--          <mesh filename="package://motoman_sia20d_support/meshes/sia20d/visual/MOTOMAN_AXIS_E.stl"/>-->
-          <mesh filename="package://reach_demo/model/motoman_sia20d/meshes/sia20d/visual/MOTOMAN_AXIS_E.stl"/>
+          <mesh filename="package://moveit_reach_plugins/demo/model/motoman_sia20d/meshes/sia20d/visual/MOTOMAN_AXIS_E.stl"/>
         </geometry>
         <material name="silver"/>
@@ -77,5 +77,5 @@
         <geometry>
 <!--          <mesh filename="package://motoman_sia20d_support/meshes/sia20d/collision/MOTOMAN_AXIS_E.stl"/>-->
-          <mesh filename="package://reach_demo/model/motoman_sia20d/meshes/sia20d/collision/MOTOMAN_AXIS_E.stl"/>
+          <mesh filename="package://moveit_reach_plugins/demo/model/motoman_sia20d/meshes/sia20d/collision/MOTOMAN_AXIS_E.stl"/>
         </geometry>
         <material name="yellow"/>
@@ -87,5 +87,5 @@
         <geometry>
 <!--          <mesh filename="package://motoman_sia20d_support/meshes/sia20d/visual/MOTOMAN_AXIS_U.stl"/>-->
-          <mesh filename="package://reach_demo/model/motoman_sia20d/meshes/sia20d/visual/MOTOMAN_AXIS_U.stl"/>
+          <mesh filename="package://moveit_reach_plugins/demo/model/motoman_sia20d/meshes/sia20d/visual/MOTOMAN_AXIS_U.stl"/>
         </geometry>
         <material name="blue"/>
@@ -95,5 +95,5 @@
         <geometry>
 <!--          <mesh filename="package://motoman_sia20d_support/meshes/sia20d/collision/MOTOMAN_AXIS_U.stl"/>-->
-          <mesh filename="package://reach_demo/model/motoman_sia20d/meshes/sia20d/collision/MOTOMAN_AXIS_U.stl"/>
+          <mesh filename="package://moveit_reach_plugins/demo/model/motoman_sia20d/meshes/sia20d/collision/MOTOMAN_AXIS_U.stl"/>
         </geometry>
         <material name="yellow"/>
@@ -105,5 +105,5 @@
         <geometry>
 <!--          <mesh filename="package://motoman_sia20d_support/meshes/sia20d/visual/MOTOMAN_AXIS_R.stl"/>-->
-          <mesh filename="package://reach_demo/model/motoman_sia20d/meshes/sia20d/visual/MOTOMAN_AXIS_R.stl"/>
+          <mesh filename="package://moveit_reach_plugins/demo/model/motoman_sia20d/meshes/sia20d/visual/MOTOMAN_AXIS_R.stl"/>
         </geometry>
         <material name="silver"/>
@@ -113,5 +113,5 @@
         <geometry>
 <!--          <mesh filename="package://motoman_sia20d_support/meshes/sia20d/collision/MOTOMAN_AXIS_R.stl"/>-->
-          <mesh filename="package://reach_demo/model/motoman_sia20d/meshes/sia20d/collision/MOTOMAN_AXIS_R.stl"/>
+          <mesh filename="package://moveit_reach_plugins/demo/model/motoman_sia20d/meshes/sia20d/collision/MOTOMAN_AXIS_R.stl"/>
         </geometry>
         <material name="yellow"/>
@@ -123,5 +123,5 @@
         <geometry>
 <!--          <mesh filename="package://motoman_sia20d_support/meshes/sia20d/visual/MOTOMAN_AXIS_B.stl"/>-->
-          <mesh filename="package://reach_demo/model/motoman_sia20d/meshes/sia20d/visual/MOTOMAN_AXIS_B.stl"/>
+          <mesh filename="package://moveit_reach_plugins/demo/model/motoman_sia20d/meshes/sia20d/visual/MOTOMAN_AXIS_B.stl"/>
         </geometry>
         <material name="blue"/>
@@ -131,5 +131,5 @@
         <geometry>
 <!--          <mesh filename="package://motoman_sia20d_support/meshes/sia20d/collision/MOTOMAN_AXIS_B.stl"/>-->
-          <mesh filename="package://reach_demo/model/motoman_sia20d/meshes/sia20d/collision/MOTOMAN_AXIS_B.stl"/>
+          <mesh filename="package://moveit_reach_plugins/demo/model/motoman_sia20d/meshes/sia20d/collision/MOTOMAN_AXIS_B.stl"/>
         </geometry>
         <material name="yellow"/>
@@ -140,5 +140,5 @@
         <geometry>
 <!--          <mesh filename="package://motoman_sia20d_support/meshes/sia20d/visual/MOTOMAN_AXIS_T.stl" />-->
-          <mesh filename="package://reach_demo/model/motoman_sia20d/meshes/sia20d/visual/MOTOMAN_AXIS_T.stl" />
+          <mesh filename="package://moveit_reach_plugins/demo/model/motoman_sia20d/meshes/sia20d/visual/MOTOMAN_AXIS_T.stl" />
         </geometry>
         <material name="silver"/>
@@ -147,5 +147,5 @@
         <geometry>
 <!--          <mesh filename="package://motoman_sia20d_support/meshes/sia20d/collision/MOTOMAN_AXIS_T.stl" />-->
-          <mesh filename="package://reach_demo/model/motoman_sia20d/meshes/sia20d/collision/MOTOMAN_AXIS_T.stl" />
+          <mesh filename="package://moveit_reach_plugins/demo/model/motoman_sia20d/meshes/sia20d/collision/MOTOMAN_AXIS_T.stl" />
         </geometry>
         <material name="yellow"/>

File: moveit_reach_plugins/demo/model/reach_study.xacro (robot description, xacro)
@@ -1,5 +1,5 @@
 <?xml version="1.0" ?>
 <robot name="reach_study" xmlns:xacro="http://ros.org/wiki/xacro">
-  <xacro:include filename="$(find reach_demo)/model/motoman_sia20d/motoman_sia20d_macro.xacro" />
+  <xacro:include filename="$(find moveit_reach_plugins)/demo/model/motoman_sia20d/motoman_sia20d_macro.xacro" />
   <xacro:motoman_sia20d prefix=""/>
   <link name="reach_object"/>
