Commit message: Updated demo files and structure

File: reach_ros/demo/model/reach_study.xacro (robot description, xacro)
@@ -3,11 +3,5 @@
   <xacro:include filename="$(find reach_ros)/demo/model/motoman_sia20d/motoman_sia20d_macro.xacro" />
   <xacro:motoman_sia20d prefix=""/>
-  <link name="reach_object"/>
   <link name="tcp"/>
-  <joint name="robot_to_reach_object" type="fixed">
-    <parent link="base_link"/>
-    <child link="reach_object"/>
-    <origin xyz="0.75 0 0.2" rpy="0 ${radians(90)} ${radians(180)}"/>
-  </joint>
   <joint name="tool0_to_tcp" type="fixed">
     <parent link="tool0"/>
